File: Hardware/BeagleboneCape-V2.sch (EAGLE design)
At the start: 11 parts, among them P8 HEADER1, P9 HEADER2

Commit message: updated V2 ( Rev B) Board to use SMD only components where possible. Using 1206 Components
Parts:
- C1, C2: device rcl:C-EU025-025X050 -> rcl:C-EUC1206
- LED1, LED2: device led:LED5MM -> led:LEDSMT1206
- R1, R2, R3: device rcl:R-EU_0207/7 -> rcl:R-EU_R1206
Connections:
- net IRQ: now also P9.28
Other:
- moved on the sheet: XB1
Changed lines of the file:
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@@
 <part name="U$9" library="microbuilder" deviceset="3.3V" device=""/>
 <part name="U$16" library="microbuilder" deviceset="GND" device=""/>
-<part name="R1" library="rcl" deviceset="R-EU_" device="0207/7" value="110R"/>
-<part name="LED1" library="led" deviceset="LED" device="5MM" value="Assoc"/>
+<part name="R1" library="rcl" deviceset="R-EU_" device="R1206" value="110R"/>
+<part name="LED1" library="led" deviceset="LED" device="SMT1206" value="Assoc"/>
 <part name="P8" library="2X23Header" deviceset="PINHD-2X24" device="" value="HEADER1"/>
 <part name="P9" library="2X23Header" deviceset="PINHD-2X24" device="" value="HEADER2"/>
@@
 <part name="U$21" library="microbuilder" deviceset="GND" device=""/>
 <part name="U$22" library="microbuilder" deviceset="GND" device=""/>
-<part name="LED2" library="led" deviceset="LED" device="5MM" value="ON_SLEEP"/>
-<part name="R2" library="rcl" deviceset="R-EU_" device="0207/7" value="110R"/>
-<part name="C1" library="rcl" deviceset="C-EU" device="025-025X050" value="1u"/>
-<part name="C2" library="rcl" deviceset="C-EU" device="025-025X050" value="8.2p"/>
-<part name="R3" library="rcl" deviceset="R-EU_" device="0207/7" value="110R"/>
+<part name="LED2" library="led" deviceset="LED" device="SMT1206" value="ON_SLEEP"/>
+<part name="R2" library="rcl" deviceset="R-EU_" device="R1206" value="110R"/>
+<part name="C1" library="rcl" deviceset="C-EU" device="C1206" value="1u"/>
+<part name="C2" library="rcl" deviceset="C-EU" device="C1206" value="8.2p"/>
+<part name="R3" library="rcl" deviceset="R-EU_" device="R1206" value="110R"/>
 <part name="U$2" library="microbuilder" deviceset="GND" device=""/>
 <part name="U$3" library="microbuilder" deviceset="3.3V" device=""/>
@@
 <pinref part="XB1" gate="G$1" pin="ASSOC/DIO5"/>
 <wire x1="116.84" y1="76.2" x2="96.52" y2="76.2" width="0.1524" layer="91"/>
-<label x="106.68" y="78.74" size="1.778" layer="95" rot="R180"/>
 <wire x1="96.52" y1="76.2" x2="96.52" y2="35.56" width="0.1524" layer="91"/>
 <pinref part="LED1" gate="G$1" pin="A"/>
@@
 <wire x1="93.98" y1="144.78" x2="81.28" y2="144.78" width="0.1524" layer="91"/>
 <label x="81.28" y="144.78" size="1.778" layer="95"/>
+</segment>
+<segment>
+<pinref part="P9" gate="A" pin="28"/>
+<wire x1="27.94" y1="35.56" x2="43.18" y2="35.56" width="0.1524" layer="91"/>
+<label x="35.56" y="35.56" size="1.778" layer="95"/>
 </segment>
 </net>
@@
 <wire x1="93.98" y1="43.18" x2="86.36" y2="43.18" width="0.1524" layer="91"/>
 <wire x1="86.36" y1="43.18" x2="86.36" y2="35.56" width="0.1524" layer="91"/>
-<label x="96.52" y="101.6" size="1.778" layer="95"/>
 <pinref part="XB1" gate="G$1" pin="ON/!SLEEP"/>
 <wire x1="116.84" y1="101.6" x2="93.98" y2="101.6" width="0.1524" layer="91"/>
