File: Hardware/Energy Sensor.sch (EAGLE design)
At the start: 0 parts

Commit message: added high power components for energy sensor. transformer needs to be sorted.
Parts:
- added C1, C2, C7: (no value), rcl:CPOL-EU140CLH-1010
- added C3, C4, C5, C6: (no value), rcl:C-EU050-025X075
- added D1: 1N4148DO35-7, diode:1N4148DO35-7
- added F1: (no value), fuse:GSH15
- added IC1: (no value), v-reg:78XXL
- added R1: P594, varistor:P594
- added R2: 100R, rcl:R-EU_0207/7
- added R3, R4, R5, R6, R7: (no value), rcl:R-EU_0207/7
- added TR1: (no value), trafo:VV11
- added U$1: CAS25-NP, CAS:CAS25-NP
- added X1, X2: (no value), con-wago-500:W237-102
Connections:
- new net +5V: C1.+, C4.1, IC1.OUT, R6.1, U$1.13
- new net CURRENT_SENSE: C5.1, R2.2
- new net GND: C1.-, C2.-, C3.2, C4.2, C5.2, C7.-, IC1.GND, R7.2, TR1.S3, U$1.12
- new net N$1: F1.1, X1-1.KL
- new net N$10: C7.+, R4.1, R6.2, R7.1
- new net N$2: R1.1, TR1.P2, X1-2.KL, X2-2.KL
- new net N$3: R2.1, U$1.11
- new net N$4: C6.2, R3.2
- new net N$5: C6.1, D1.A, TR1.S4
- new net N$6: F1.2, R1.2, TR1.P1, U$1.1, U$1.2, U$1.3
- new net N$7: C2.+, C3.1, D1.C, IC1.IN
- new net N$8: U$1.10, U$1.8, U$1.9, X2-1.KL
- new net N$9: R3.1, R4.2, R5.2
- new net VSENSE: R5.1
