File: Hardware/Energy Sensor.sch (EAGLE design)
At the start: 42 parts, among them IC1 7805, IC2 ATMega328p-pu, IC3 ld33v, Q1 16MHz, X1 MAINS IN, X2 MAINS OUT

Commit message: updated to fuse and varistor arrangements
Other:
- moved on the sheet: F1
Changed lines of the file:
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@@
 <?xml version="1.0" encoding="utf-8"?>
 <!DOCTYPE eagle SYSTEM "eagle.dtd">
-<eagle version="6.5.0">
+<eagle version="6.4">
 <drawing>
 <settings>
@@
 <instance part="X2" gate="-2" x="-20.32" y="22.86"/>
 <instance part="R1" gate="1" x="35.56" y="76.2" rot="R90"/>
-<instance part="F1" gate="1" x="12.7" y="76.2" rot="R90"/>
+<instance part="F1" gate="1" x="12.7" y="68.58" rot="R90"/>
 <instance part="TR1" gate="1" x="45.72" y="78.74"/>
 <instance part="D1" gate="G$1" x="68.58" y="83.82"/>
@@
 <wire x1="25.4" y1="60.96" x2="25.4" y2="63.5" width="0.1524" layer="91"/>
 <wire x1="25.4" y1="63.5" x2="30.48" y2="63.5" width="0.1524" layer="91"/>
-<wire x1="12.7" y1="71.12" x2="12.7" y2="63.5" width="0.1524" layer="91"/>
 <wire x1="25.4" y1="63.5" x2="12.7" y2="63.5" width="0.1524" layer="91"/>
 <junction x="25.4" y="63.5"/>
@@
 <pinref part="F2" gate="1" pin="1"/>
 <wire x1="15.24" y1="83.82" x2="12.7" y2="83.82" width="0.1524" layer="91"/>
-<wire x1="12.7" y1="83.82" x2="12.7" y2="81.28" width="0.1524" layer="91"/>
+<wire x1="12.7" y1="83.82" x2="12.7" y2="73.66" width="0.1524" layer="91"/>
 <pinref part="F1" gate="1" pin="2"/>
 <wire x1="-15.24" y1="83.82" x2="12.7" y2="83.82" width="0.1524" layer="91"/>

Commit message: updated wrong fuse holder and incorrect terminal and processor mounts
Parts:
- F1, F2: device fuse:GSH15 -> fuse:SH22,5A
- IC2: device ic-package:DIL28-4 -> ic-package:DIL28-3
Connections:
- net N$2: now also X1-1.KL, X2-2.KL; no longer X1-2.KL, X2-1.KL
- net N$22: now also X1-2.KL; no longer X1-1.KL
- net N$8: now also X2-1.KL; no longer X2-2.KL
Changed lines of the file:
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@@
 <part name="X2" library="con-wago-500" deviceset="W237-102" device="" value="MAINS OUT"/>
 <part name="R1" library="varistor" deviceset="P594" device=""/>
-<part name="F1" library="fuse" deviceset="GSH15" device="" value="230V 10A"/>
+<part name="F1" library="fuse" deviceset="SH22,5A" device="" value="230V 10A"/>
 <part name="TR1" library="xformer" deviceset="VV11" device="" value="vn20.10 09477"/>
 <part name="D1" library="diode" deviceset="1N4148" device="DO35-7"/>
@@
 <part name="R7" library="rcl" deviceset="R-EU_" device="0207/7" value="470k"/>
 <part name="GND3" library="supply1" deviceset="GND" device=""/>
-<part name="IC2" library="ic-package" deviceset="DIL28" device="-4" value="ATMega328p-pu"/>
+<part name="IC2" library="ic-package" deviceset="DIL28" device="-3" value="ATMega328p-pu"/>
 <part name="GND4" library="supply1" deviceset="GND" device=""/>
 <part name="Q1" library="crystal" deviceset="CRYSTAL" device="HC49S" value="16MHz"/>
@@
 <part name="H3" library="holes" deviceset="MOUNT-HOLE" device="2.8"/>
 <part name="H4" library="holes" deviceset="MOUNT-HOLE" device="2.8"/>
-<part name="F2" library="fuse" deviceset="GSH15" device="" value="230V 100mA"/>
+<part name="F2" library="fuse" deviceset="SH22,5A" device="" value="230V 100mA"/>
 </parts>
 <sheets>
@@
 <net name="N$2" class="0">
 <segment>
-<wire x1="5.08" y1="73.66" x2="5.08" y2="68.58" width="0.1524" layer="91"/>
 <wire x1="5.08" y1="68.58" x2="30.48" y2="68.58" width="0.1524" layer="91"/>
-<wire x1="5.08" y1="68.58" x2="5.08" y2="27.94" width="0.1524" layer="91"/>
+<wire x1="5.08" y1="68.58" x2="5.08" y2="22.86" width="0.1524" layer="91"/>
 <wire x1="30.48" y1="68.58" x2="30.48" y2="71.12" width="0.1524" layer="91"/>
 <junction x="5.08" y="68.58"/>
-<pinref part="X2" gate="-1" pin="KL"/>
-<wire x1="-15.24" y1="27.94" x2="5.08" y2="27.94" width="0.1524" layer="91"/>
 <pinref part="TR1" gate="1" pin="P2"/>
 <wire x1="30.48" y1="71.12" x2="35.56" y2="71.12" width="0.1524" layer="91"/>
@@
 <wire x1="35.56" y1="71.12" x2="40.64" y2="71.12" width="0.1524" layer="91"/>
 <junction x="35.56" y="71.12"/>
-<pinref part="X1" gate="-2" pin="KL"/>
-<wire x1="-15.24" y1="73.66" x2="5.08" y2="73.66" width="0.1524" layer="91"/>
+<pinref part="X1" gate="-1" pin="KL"/>
+<wire x1="-15.24" y1="78.74" x2="5.08" y2="78.74" width="0.1524" layer="91"/>
+<wire x1="5.08" y1="78.74" x2="5.08" y2="68.58" width="0.1524" layer="91"/>
+<pinref part="X2" gate="-2" pin="KL"/>
+<wire x1="5.08" y1="22.86" x2="-15.24" y2="22.86" width="0.1524" layer="91"/>
 </segment>
 </net>
@@
 <wire x1="25.4" y1="27.94" x2="30.48" y2="27.94" width="0.1524" layer="91"/>
 <junction x="30.48" y="27.94"/>
-<pinref part="X2" gate="-2" pin="KL"/>
-<wire x1="-15.24" y1="22.86" x2="30.48" y2="22.86" width="0.1524" layer="91"/>
 <wire x1="30.48" y1="22.86" x2="30.48" y2="27.94" width="0.1524" layer="91"/>
+<pinref part="X2" gate="-1" pin="KL"/>
+<wire x1="-15.24" y1="27.94" x2="10.16" y2="27.94" width="0.1524" layer="91"/>
+<wire x1="10.16" y1="27.94" x2="10.16" y2="22.86" width="0.1524" layer="91"/>
+<wire x1="10.16" y1="22.86" x2="30.48" y2="22.86" width="0.1524" layer="91"/>
 </segment>
 </net>
@@
 <net name="N$22" class="0">
 <segment>
-<pinref part="X1" gate="-1" pin="KL"/>
-<wire x1="-15.24" y1="78.74" x2="-15.24" y2="83.82" width="0.1524" layer="91"/>
 <pinref part="F2" gate="1" pin="1"/>
 <wire x1="15.24" y1="83.82" x2="12.7" y2="83.82" width="0.1524" layer="91"/>
 <wire x1="12.7" y1="83.82" x2="12.7" y2="73.66" width="0.1524" layer="91"/>
 <pinref part="F1" gate="1" pin="2"/>
-<wire x1="-15.24" y1="83.82" x2="12.7" y2="83.82" width="0.1524" layer="91"/>
 <junction x="12.7" y="83.82"/>
-</segment>
-</net>
+<pinref part="X1" gate="-2" pin="KL"/>
+<wire x1="-7.62" y1="83.82" x2="12.7" y2="83.82" width="0.1524" layer="91"/>
+<wire x1="-15.24" y1="73.66" x2="-7.62" y2="73.66" width="0.1524" layer="91"/>
+<wire x1="-7.62" y1="73.66" x2="-7.62" y2="83.82" width="0.1524" layer="91"/>
+</segment>
+</net>
