File: Hardware/Environment Sensor.sch (EAGLE design)
At the start: 0 parts

Commit message: added basic components still awaiting Vreg and sensor devices
Parts:
- added C1, C2, C3: (no value), rcl:C-EUC1206K
- added G1: CR2032H, battery:CR2032H
- added IC1: ATMEGA644A, atmel:ATMEGA644A
- added Q1: (no value), crystal:CRYSTALHC49UP
- added R2: (no value), rcl:R-EU_R1206
- added U$1: 2X4SMDHEADER, Header:2X4SMDHEADER
Connections:
- new net CE_RAD: U$1.3
- new net CSN_RAD: U$1.4
- new net GND: C1.2, C2.2, C3.2, G1.-, IC1.GND, IC1.GND@1, IC1.GND@2, IC1.GND@3, U$1.1
- new net IRQ_RAD: U$1.8
- new net MISO: IC1.(PCINT14/MISO)PB6, U$1.7
- new net MOSI: U$1.6
- new net MSOI: IC1.(PCINT13/MOSI)PB5
- new net N$1: C1.1, IC1.XTAL2, Q1.1
- new net N$2: C2.1, IC1.XTAL1, Q1.2
- new net N$3: IC1.RESET, R2.2
- new net N$4: IC1.(PCINT11/OC0A/AIN1)PB3
- new net N$5: IC1.(PCINT10/INT2/AIN0)PB2
- new net N$7: IC1.(PCINT12/OC0B/!SS!)PB4
- new net SCK: IC1.(PCINT15/SCK)PB7, U$1.5
- new net VCC: C3.1, G1.+, IC1.VCC, IC1.VCC@1, IC1.VCC@2, R2.1, U$1.2
