File: Hardware/Energy Sensor.brd (EAGLE design)
At the start: 159 x 63 mm, 42 parts, among them IC1 7805, IC2 ATMega328p-pu, IC3 ld33v, Q1 16MHz, X1 MAINS IN, X2 MAINS OUT

Commit message: updated wrong fuse holder and incorrect terminal and processor mounts
Parts:
- F1, F2: device fuse:GSH15 -> fuse:SH22,5A
- IC2: device ic-package:DIL28-4 -> ic-package:DIL28-3
- moved F2 3.00 mm to (34.0, 22.0)
- moved X1 1.87 mm to (11.6, 22.2), turned to 270 degrees
- moved X2 1.83 mm to (12.4, 44.3), turned to 270 degrees
Connections:
- net N$2: now also X1.1, X2.2; no longer X1.2, X2.1
- net N$22: now also X1.2; no longer X1.1
- net N$8: now also X2.1; no longer X2.2
Routing:
- net N$19: track 24.6 -> 32.2 mm
- net N$6: track 38.3 -> 43.5 mm
- net N$2: track 103.4 -> 100.8 mm
- net N$22: track 25.2 -> 27.3 mm
- net +3V3: track 121.9 -> 120.3 mm
- net INT: track 39.3 -> 38.0 mm
- net CE: track 25.9 -> 27.2 mm
- net N$13: track 8.76 -> 10.0 mm
- net N$12: track 10.0 -> 11.3 mm
- net MOSI: track 38.2 -> 36.9 mm
- net MISO: track 40.2 -> 41.4 mm
- net CURRENT_SENSE: track 89.6 -> 90.9 mm
- net CSN: track 25.9 -> 27.2 mm
- net SCK: track 40.2 -> 41.4 mm
- net N$18: track 9.58 -> 10.8 mm
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