File: Hardware/Power Outlet-RevB.sch (EAGLE design)
At the start: 38 parts, among them IC1 ATMega 328p-pu, IC2 ULN2003AD, K1 G5LE, K2 G5LE, Q1 8MHz, X1 VIN, X2 VOUT2, X3 VOUT1, X7 EARTH

Commit message: updated wrong capacitor footprint, removed isolation cap as causes circuit not to function.
Parts:
- removed C6: 1n/2Kv, rcl:C-EUC1206K
- added D1: (no value), diode:SCHOTTKY-DIODESMC
- C2: device rcl:C-EU050-030X075 -> rcl:C-EU150-054X183
Connections:
- removed net AGND: C6.2, IC2.GND, IC2.I5, IC2.I6, IC2.I7
- net +3V3: now also D1.C
- net GND: now also D1.A, IC2.GND, IC2.I5, IC2.I6, IC2.I7; no longer C6.1
Changed lines of the file:
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@@
 <part name="+3V1" library="supply1" deviceset="+3V3" device=""/>
 <part name="GND1" library="supply1" deviceset="GND" device=""/>
-<part name="C2" library="rcl" deviceset="C-EU" device="050-030X075" value="0.1u/275V"/>
+<part name="C2" library="rcl" deviceset="C-EU" device="150-054X183" value="0.1u/275V"/>
 <part name="K1" library="relay" deviceset="G5LE" device=""/>
 <part name="K2" library="relay" deviceset="G5LE" device=""/>
@@
 <part name="SUPPLY2" library="supply2" deviceset="VCC" device=""/>
 <part name="L1" library="rcl" deviceset="L-EU" device="L3225P"/>
-<part name="C6" library="rcl" deviceset="C-EU" device="C1206K" value="1n/2Kv"/>
-<part name="SUPPLY3" library="supply2" deviceset="AGND" device=""/>
-<part name="SUPPLY4" library="supply2" deviceset="AGND" device=""/>
 <part name="SUPPLY5" library="supply2" deviceset="VCC" device=""/>
 <part name="R7" library="rcl" deviceset="R-EU_" device="R1206W" value="100R"/>
@@
 <part name="EARTH1" library="supply2" deviceset="GND1" device=""/>
 <part name="L2" library="rcl" deviceset="L-EU" device="L3225P"/>
+<part name="D1" library="diode" deviceset="SCHOTTKY-DIODE" device="SMC"/>
+<part name="GND6" library="supply1" deviceset="GND" device=""/>
 </parts>
 <sheets>
@@
 <instance part="SUPPLY2" gate="G$1" x="93.98" y="81.28"/>
 <instance part="L1" gate="G$1" x="86.36" y="76.2" rot="R90"/>
-<instance part="C6" gate="G$1" x="86.36" y="60.96" rot="R90"/>
-<instance part="SUPPLY3" gate="G$1" x="157.48" y="0"/>
-<instance part="SUPPLY4" gate="G$1" x="93.98" y="55.88"/>
 <instance part="SUPPLY5" gate="G$1" x="193.04" y="48.26"/>
 <instance part="R7" gate="G$1" x="134.62" y="35.56" rot="R180"/>
@@
 <instance part="EARTH1" gate="G$1" x="-71.12" y="-10.16"/>
 <instance part="L2" gate="G$1" x="60.96" y="76.2" rot="R90"/>
+<instance part="D1" gate="G$1" x="53.34" y="68.58" rot="R90"/>
+<instance part="GND6" gate="1" x="157.48" y="0"/>
 </instances>
 <busses>
@@
 <wire x1="55.88" y1="76.2" x2="53.34" y2="76.2" width="0.1524" layer="91"/>
 <wire x1="53.34" y1="76.2" x2="50.8" y2="73.66" width="0.1524" layer="91"/>
+<pinref part="D1" gate="G$1" pin="C"/>
+<wire x1="53.34" y1="71.12" x2="53.34" y2="76.2" width="0.1524" layer="91"/>
+<junction x="53.34" y="76.2"/>
 </segment>
 </net>
@@
 <wire x1="76.2" y1="66.04" x2="76.2" y2="60.96" width="0.1524" layer="91"/>
 <junction x="76.2" y="60.96"/>
-<junction x="78.74" y="60.96"/>
-<pinref part="C6" gate="G$1" pin="1"/>
-<wire x1="83.82" y1="60.96" x2="78.74" y2="60.96" width="0.1524" layer="91"/>
 <pinref part="U$1" gate="G$1" pin="GND"/>
 <wire x1="68.58" y1="60.96" x2="53.34" y2="60.96" width="0.1524" layer="91"/>
 <wire x1="53.34" y1="60.96" x2="50.8" y2="63.5" width="0.1524" layer="91"/>
 <junction x="68.58" y="60.96"/>
+<pinref part="D1" gate="G$1" pin="A"/>
+<wire x1="53.34" y1="66.04" x2="53.34" y2="60.96" width="0.1524" layer="91"/>
+<junction x="53.34" y="60.96"/>
 </segment>
 <segment>
@@
 <junction x="104.14" y="12.7"/>
 </segment>
+<segment>
+<pinref part="IC2" gate="A" pin="GND"/>
+<wire x1="160.02" y1="7.62" x2="157.48" y2="7.62" width="0.1524" layer="91"/>
+<pinref part="IC2" gate="A" pin="I5"/>
+<wire x1="160.02" y1="15.24" x2="157.48" y2="15.24" width="0.1524" layer="91"/>
+<wire x1="157.48" y1="15.24" x2="157.48" y2="12.7" width="0.1524" layer="91"/>
+<pinref part="IC2" gate="A" pin="I6"/>
+<wire x1="157.48" y1="12.7" x2="157.48" y2="10.16" width="0.1524" layer="91"/>
+<wire x1="157.48" y1="10.16" x2="157.48" y2="7.62" width="0.1524" layer="91"/>
+<wire x1="160.02" y1="12.7" x2="157.48" y2="12.7" width="0.1524" layer="91"/>
+<pinref part="IC2" gate="A" pin="I7"/>
+<wire x1="160.02" y1="10.16" x2="157.48" y2="10.16" width="0.1524" layer="91"/>
+<junction x="157.48" y="12.7"/>
+<junction x="157.48" y="10.16"/>
+<junction x="157.48" y="7.62"/>
+<wire x1="157.48" y1="2.54" x2="157.48" y2="7.62" width="0.1524" layer="91"/>
+<pinref part="GND6" gate="1" pin="GND"/>
+</segment>
 </net>
 <net name="N$4" class="0">
@@
 </segment>
 </net>
-<net name="AGND" class="0">
-<segment>
-<pinref part="SUPPLY4" gate="G$1" pin="AGND"/>
-<pinref part="C6" gate="G$1" pin="2"/>
-<wire x1="93.98" y1="58.42" x2="93.98" y2="60.96" width="0.1524" layer="91"/>
-<wire x1="93.98" y1="60.96" x2="91.44" y2="60.96" width="0.1524" layer="91"/>
-</segment>
-<segment>
-<pinref part="IC2" gate="A" pin="GND"/>
-<wire x1="160.02" y1="7.62" x2="157.48" y2="7.62" width="0.1524" layer="91"/>
-<pinref part="IC2" gate="A" pin="I5"/>
-<wire x1="160.02" y1="15.24" x2="157.48" y2="15.24" width="0.1524" layer="91"/>
-<wire x1="157.48" y1="15.24" x2="157.48" y2="12.7" width="0.1524" layer="91"/>
-<pinref part="IC2" gate="A" pin="I6"/>
-<wire x1="157.48" y1="12.7" x2="157.48" y2="10.16" width="0.1524" layer="91"/>
-<wire x1="157.48" y1="10.16" x2="157.48" y2="7.62" width="0.1524" layer="91"/>
-<wire x1="160.02" y1="12.7" x2="157.48" y2="12.7" width="0.1524" layer="91"/>
-<pinref part="IC2" gate="A" pin="I7"/>
-<wire x1="160.02" y1="10.16" x2="157.48" y2="10.16" width="0.1524" layer="91"/>
-<junction x="157.48" y="12.7"/>
-<junction x="157.48" y="10.16"/>
-<junction x="157.48" y="7.62"/>
-<pinref part="SUPPLY3" gate="G$1" pin="AGND"/>
-<wire x1="157.48" y1="2.54" x2="157.48" y2="7.62" width="0.1524" layer="91"/>
-</segment>
-</net>
