File: Hardware/Connections/PoE.brd (EAGLE design)
At the start: 34.3 x 28.9 mm, 4 parts

Commit message: updated PoE Schematic slightly and added eagle project file. Updated Readme to explain current directory structure
Parts:
- added C1: 10nF, rcl:C1206
- added C2: 4.7uF, rcl:C1206
- added C3, C4: 18p, rcl:C1206
- added C5: 0.1u, rcl:C1206
- added C6: 10uF/16V, rcl:140CLH-1010
- added Q1: 25MHz, crystal:HC49UP
- added R10, R11, R12, R13, R14, R15, R7, R8, R9: 77k, resistor:R1206
- added R3: 1M, resistor:R1206
- added R4, R5, R6: (no value), resistor:R1206
- added U1: W5500, W5500:W5500
Connections:
- new net ACTLED: U1.27
- new net LINKLED: U1.25
- new net N$1: R9.1, U1.43
- new net N$10: R14.1, U1.39
- new net N$11: R11.1, U1.40
- new net N$12: R12.1, U1.41
- new net N$13: R13.1, U1.42
- new net N$2: C1.1, U1.22
- new net N$3: C2.1, U1.20
- new net N$4: C4.1, Q1.1, R3.1
- new net N$5: C3.1, Q1.2, U1.30
- new net N$6: R7.1, U1.44
- new net N$7: R3.2, U1.31
- new net N$8: R8.1, U1.45
- new net N$9: R15.1, U1.38
- new net RESET: R10.1, U1.37
- net +3V3: now also C5.1, C6.+, R10.2, R7.2, R8.2, R9.2, U1.11, U1.15, U1.17, U1.21, U1.28, U1.4, U1.8
- net CSN_RAD: now also U1.32
- net GND: now also C1.2, C2.2, C3.2, C4.2, C5.2, C6.-, R11.2, R12.2, R13.2, R14.2, R15.2, U1.14, U1.16, U1.19, U1.29, U1.3, U1.48, U1.9
- net IRQ_RAD: now also U1.36
- net MISO: now also U1.34
- net MOSI: now also U1.35
- net SCK: now also U1.33

Commit message: updated POE design. missing power circuitry and suitable rj45 connector
Parts:
- added C10, C11: 6.8, rcl:C1206
- added C12, C13, C14, C15, C16, C17: 0.1u, rcl:C1206
- added C18: 10uF/16V, rcl:153CLV-0405
- added C7: 1nF/2kV, rcl:C1206
- added C8: 22n, rcl:C1206
- added C9: 10n, rcl:C1206
- added L1: (no value), inductor-neosid:MS50
- added R16, R17: 49R9 1%, resistor:R1206
- added R18: 12.4k 1%, resistor:R1206
- added R19, R20: 330R, resistor:R1206
- C6: device rcl:140CLH-1010 -> rcl:153CLV-0505
- R4, R5: value (none) -> 49R9 1%
- R6: value (none) -> 10R 1%
Connections:
- new net GNDA: C7.2
- new net N$14: R5.1, U1.2
- new net N$16: C8.1, R6.1
- new net N$17: R4.1, U1.1
- new net N$18: C10.1, R16.2, U1.6
- new net N$19: C9.1, R16.1, R17.1
- new net N$20: C11.2
- new net N$21: C10.2
- new net N$22: R18.2, U1.10
- new net VDD: C12.1, C13.1, C14.1, C15.1, C16.1, C17.1, C18.+, L1.2, R4.2, R5.2, R6.2, U1.11, U1.15, U1.17, U1.21, U1.4, U1.8
- net +3V3: now also L1.1; no longer U1.11, U1.15, U1.17, U1.21, U1.4, U1.8
- net GND: now also C1.1, C12.2, C13.2, C14.2, C15.2, C16.2, C17.2, C18.-, C7.1, C8.2, C9.2, R18.1; no longer C1.2
- net N$2: now also C1.2; no longer C1.1
- net N$4: now also U1.31
- net N$5: now also R3.2
- net N$7: now also C11.1, R17.2, U1.5; no longer R3.2, U1.31
