File: Hardware/EnvironmentSensor/Environment Sensor.sch (EAGLE design)
At the start: 18 parts, among them IC1 ATMEGA328P-AU, Q1 8MHz

Commit message: updated component Values
Parts:
- C3: value 0.1u -> 1u
- C4: value (none) -> 100n
Changed lines of the file:
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@@
 <part name="P+3" library="supply1" deviceset="VCC" device=""/>
 <part name="GND4" library="supply1" deviceset="GND" device=""/>
-<part name="C3" library="rcl" deviceset="C-EU" device="C1206K" value="0.1u"/>
+<part name="C3" library="rcl" deviceset="C-EU" device="C1206K" value="1u"/>
 <part name="P+4" library="supply1" deviceset="VCC" device=""/>
 <part name="L1" library="rcl" deviceset="L-EU" device="L3216C" value="10u"/>
-<part name="C4" library="rcl" deviceset="C-EU" device="C1206"/>
+<part name="C4" library="rcl" deviceset="C-EU" device="C1206" value="100n"/>
 <part name="GND5" library="supply1" deviceset="GND" device=""/>
 <part name="G2" library="battery" deviceset="SL-160AA/PR" device=""/>
