File: Hardware/EnergySensor/Energy SensorRevB.brd (EAGLE design)
At the start: 156 x 54 mm, 42 parts, among them IC2 ATMega328p-pu, IC3 ld33v, Q1 16MHz, X1 MAINS IN

Commit message: FIXED MAJOR BUG  - schematic was incorrect for power measurements
Parts:
- removed C13: 1u, rcl:C1206K
- R4: device rcl:0207/7 -> rcl:R1206
- moved R4 9.76 mm to (82.0, 12.3), flipped to the bottom, turned to 270 degrees
Connections:
- removed net N$10: C10.1, C13.2, R5.2, R6.2, R7.1
- new net N$11: C10.1, R4.1, R6.2, R7.1
- net GND: no longer R4.1
- net N$9: now also R5.2; no longer C13.1
Routing:
- net N$10: track 31.4 -> 0.00 mm
- net N$9: track 7.49 -> 32.4 mm
- net N$11: track 0.00 -> 12.1 mm
Changed lines of the file:
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@@
 <grid distance="1" unitdist="mm" unit="mm" style="lines" multiple="1" display="no" altdistance="0.05" altunitdist="mm" altunit="mm"/>
 <layers>
-<layer number="1" name="Top" color="4" fill="1" visible="no" active="yes"/>
+<layer number="1" name="Top" color="4" fill="1" visible="yes" active="yes"/>
 <layer number="2" name="Route2" color="1" fill="3" visible="no" active="no"/>
 <layer number="3" name="Route3" color="4" fill="3" visible="no" active="no"/>
@@
 <layer number="14" name="Route14" color="1" fill="6" visible="no" active="no"/>
 <layer number="15" name="Route15" color="4" fill="6" visible="no" active="no"/>
-<layer number="16" name="Bottom" color="1" fill="1" visible="no" active="yes"/>
-<layer number="17" name="Pads" color="2" fill="1" visible="no" active="yes"/>
-<layer number="18" name="Vias" color="2" fill="1" visible="no" active="yes"/>
-<layer number="19" name="Unrouted" color="6" fill="1" visible="no" active="yes"/>
+<layer number="16" name="Bottom" color="1" fill="1" visible="yes" active="yes"/>
+<layer number="17" name="Pads" color="2" fill="1" visible="yes" active="yes"/>
+<layer number="18" name="Vias" color="2" fill="1" visible="yes" active="yes"/>
+<layer number="19" name="Unrouted" color="6" fill="1" visible="yes" active="yes"/>
 <layer number="20" name="Dimension" color="15" fill="1" visible="yes" active="yes"/>
 <layer number="21" name="tPlace" color="7" fill="1" visible="yes" active="yes"/>
 <layer number="22" name="bPlace" color="7" fill="1" visible="yes" active="yes"/>
-<layer number="23" name="tOrigins" color="15" fill="1" visible="no" active="yes"/>
-<layer number="24" name="bOrigins" color="15" fill="1" visible="no" active="yes"/>
+<layer number="23" name="tOrigins" color="15" fill="1" visible="yes" active="yes"/>
+<layer number="24" name="bOrigins" color="15" fill="1" visible="yes" active="yes"/>
 <layer number="25" name="tNames" color="7" fill="1" visible="yes" active="yes"/>
-<layer number="26" name="bNames" color="7" fill="1" visible="no" active="yes"/>
-<layer number="27" name="tValues" color="7" fill="1" visible="no" active="yes"/>
-<layer number="28" name="bValues" color="7" fill="1" visible="no" active="yes"/>
-<layer number="29" name="tStop" color="7" fill="3" visible="no" active="yes"/>
-<layer number="30" name="bStop" color="7" fill="6" visible="no" active="yes"/>
+<layer number="26" name="bNames" color="7" fill="1" visible="yes" active="yes"/>
+<layer number="27" name="tValues" color="7" fill="1" visible="yes" active="yes"/>
+<layer number="28" name="bValues" color="7" fill="1" visible="yes" active="yes"/>
+<layer number="29" name="tStop" color="7" fill="3" visible="yes" active="yes"/>
+<layer number="30" name="bStop" color="7" fill="6" visible="yes" active="yes"/>
 <layer number="31" name="tCream" color="7" fill="4" visible="no" active="yes"/>
 <layer number="32" name="bCream" color="7" fill="5" visible="no" active="yes"/>
@@
 <element name="C6" library="rcl" package="C1206K" value="1u" x="75.07" y="18.88" rot="MR270"/>
 <element name="R3" library="rcl" package="0207/7" value="120K" x="78.18" y="8.37" rot="R180"/>
-<element name="R4" library="rcl" package="0207/7" value="10k" x="78.16" y="3.38"/>
+<element name="R4" library="rcl" package="R1206" value="10k" x="82.02" y="12.34" rot="MR270"/>
 <element name="R5" library="rcl" package="0207/7" value="1k" x="97.15" y="26.37" smashed="yes" rot="R180">
 <attribute name="NAME" x="96.69" y="28.973" size="1.27" layer="25" ratio="10" rot="R180"/>
@@
 <element name="R9" library="rcl" package="0207/7" value="330R" x="138.74" y="14.27" rot="R90"/>
 <element name="R10" library="rcl" package="0207/7" value="330R" x="135.01" y="12.03" rot="R90"/>
-<element name="C13" library="rcl" package="C1206K" value="1u" x="81.93" y="12.34" rot="MR90"/>
 <element name="JP1" library="jumper" package="JP1" value="Extern_Power" x="75.58" y="26.55" smashed="yes">
 <attribute name="NAME" x="76.929" y="30.01" size="1.27" layer="25" ratio="10" rot="R90"/>
@@
 <contactref element="R7" pad="2"/>
 <contactref element="C10" pad="2"/>
-<contactref element="R4" pad="1"/>
 <contactref element="IC2" pad="8"/>
 <contactref element="C8" pad="2"/>
@@
 <contactref element="R3" pad="1"/>
 <contactref element="R4" pad="2"/>
-<contactref element="C13" pad="1"/>
-<wire x1="81.97" y1="3.38" x2="81.97" y2="8.35" width="1.016" layer="16"/>
 <wire x1="81.97" y1="8.35" x2="81.99" y2="8.37" width="1.016" layer="16"/>
-<wire x1="81.99" y1="8.37" x2="81.99" y2="10.78" width="1.016" layer="16"/>
-<wire x1="81.99" y1="10.78" x2="81.93" y2="10.84" width="1.016" layer="16"/>
+<contactref element="R5" pad="2"/>
+<wire x1="93.34" y1="26.37" x2="93.34" y2="17.34" width="1.016" layer="16"/>
+<wire x1="93.34" y1="17.34" x2="91" y2="15" width="1.016" layer="16"/>
+<wire x1="91" y1="15" x2="91" y2="9" width="1.016" layer="16"/>
+<wire x1="91" y1="9" x2="88" y2="6" width="1.016" layer="16"/>
+<wire x1="88" y1="6" x2="84" y2="6" width="1.016" layer="16"/>
+<wire x1="84" y1="6" x2="81.99" y2="8.01" width="1.016" layer="16"/>
+<wire x1="81.99" y1="8.01" x2="81.99" y2="8.37" width="1.016" layer="16"/>
+<wire x1="81.99" y1="8.37" x2="82.02" y2="8.4" width="1.016" layer="16"/>
+<wire x1="82.02" y1="8.4" x2="82.02" y2="10.918" width="1.016" layer="16"/>
 </signal>
 <signal name="VSENSE">
@@
 <wire x1="131.71" y1="15.84" x2="135.01" y2="15.84" width="1.016" layer="16"/>
 </signal>
-<signal name="N$10">
-<contactref element="R6" pad="2"/>
-<contactref element="C13" pad="2"/>
-<contactref element="R7" pad="1"/>
-<contactref element="R5" pad="2"/>
-<contactref element="C10" pad="1"/>
-<wire x1="84.71" y1="10.59" x2="84.71" y2="13" width="1.016" layer="16"/>
-<wire x1="84.71" y1="13" x2="84.71" y2="13.29" width="1.016" layer="16"/>
-<wire x1="84.71" y1="13.29" x2="84" y2="14" width="1.016" layer="16"/>
-<wire x1="84" y1="14" x2="82.09" y2="14" width="1.016" layer="16"/>
-<wire x1="82.09" y1="14" x2="81.93" y2="13.84" width="1.016" layer="16"/>
-<wire x1="77.93" y1="16.91" x2="80.32" y2="16.91" width="1.016" layer="16"/>
-<wire x1="80.32" y1="16.91" x2="80.63" y2="16.6" width="1.016" layer="16"/>
-<wire x1="80.63" y1="16.6" x2="80.63" y2="15.14" width="1.016" layer="16"/>
-<wire x1="80.63" y1="15.14" x2="81.93" y2="13.84" width="1.016" layer="16"/>
-<wire x1="93.34" y1="26.37" x2="93.34" y2="17.34" width="1.016" layer="16"/>
-<wire x1="93.34" y1="17.34" x2="93" y2="17" width="1.016" layer="16"/>
-<wire x1="93" y1="17" x2="88.71" y2="17" width="1.016" layer="16"/>
-<wire x1="88.71" y1="17" x2="84.71" y2="13" width="1.016" layer="16"/>
-</signal>
 <signal name="N$20">
 <via x="151" y="42" extent="1-16" drill="0.6" diameter="1.778"/>
@@
 <wire x1="120.5" y1="35.55" x2="119.6" y2="37" width="1.016" layer="16"/>
 </signal>
+<signal name="N$11">
+<contactref element="R4" pad="1"/>
+<contactref element="R6" pad="2"/>
+<contactref element="R7" pad="1"/>
+<contactref element="C10" pad="1"/>
+<wire x1="84.71" y1="13.29" x2="84" y2="14" width="1.016" layer="16"/>
+<wire x1="84" y1="14" x2="82.09" y2="14" width="1.016" layer="16"/>
+<wire x1="77.93" y1="16.91" x2="80.32" y2="16.91" width="1.016" layer="16"/>
+<wire x1="80.32" y1="16.91" x2="80.63" y2="16.6" width="1.016" layer="16"/>
+<wire x1="80.63" y1="16.6" x2="80.63" y2="15.14" width="1.016" layer="16"/>
+<wire x1="80.63" y1="15.14" x2="80.95" y2="15.14" width="1.016" layer="16"/>
+<wire x1="80.95" y1="15.14" x2="82.045" y2="14.045" width="1.016" layer="16"/>
+<wire x1="82.045" y1="14.045" x2="82.09" y2="14" width="1.016" layer="16"/>
+<wire x1="82.02" y1="13.762" x2="82.02" y2="14.02" width="1.016" layer="16"/>
+<wire x1="82.02" y1="14.02" x2="82.045" y2="14.045" width="1.016" layer="16"/>
+<wire x1="84.71" y1="10.59" x2="84.71" y2="13.29" width="1.016" layer="16"/>
+</signal>
 </signals>

Commit message: updated BOM with finalised pricelist
Parts:
- C11, C4: value 10u -> 47u
- R10, R9: value 330R -> 3k3
Changed lines of the file:
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@@
 <attribute name="VALUE" x="83.723" y="38.89" size="1.778" layer="27" ratio="10"/>
 </element>
-<element name="C11" library="rcl" package="E3,5-8" value="10u" x="99.29" y="43.23" rot="R180"/>
+<element name="C11" library="rcl" package="E3,5-8" value="47u" x="99.29" y="43.23" rot="R180"/>
 <element name="C12" library="rcl" package="C025-025X050" value="1n" x="89.23" y="25.93"/>
 <element name="LINK" library="led" package="LED5MM" value="GRN" x="143.85" y="10.69"/>
@@
 <attribute name="VALUE" x="146.9704" y="16.7766" size="1.27" layer="27" ratio="10"/>
 </element>
-<element name="R9" library="rcl" package="0207/7" value="330R" x="138.74" y="14.27" rot="R90"/>
-<element name="R10" library="rcl" package="0207/7" value="330R" x="135.01" y="12.03" rot="R90"/>
+<element name="R9" library="rcl" package="0207/7" value="3k3" x="138.74" y="14.27" rot="R90"/>
+<element name="R10" library="rcl" package="0207/7" value="3k3" x="135.01" y="12.03" rot="R90"/>
 <element name="JP1" library="jumper" package="JP1" value="Extern_Power" x="75.58" y="26.55" smashed="yes">
 <attribute name="NAME" x="76.929" y="30.01" size="1.27" layer="25" ratio="10" rot="R90"/>
@@
 <attribute name="VALUE" x="99.5588" y="17.714" size="1.27" layer="27" ratio="10" rot="R90"/>
 </element>
-<element name="C4" library="rcl" package="E3,5-8" value="10u" x="139" y="41"/>
+<element name="C4" library="rcl" package="E3,5-8" value="47u" x="139" y="41"/>
 <element name="C5" library="rcl" package="C1206K" value="100n" x="119" y="34" smashed="yes" rot="MR0">
 <attribute name="NAME" x="115.6" y="36.1" size="1.016" layer="26" rot="MR0"/>
